File: COdetector_pcb/PCB_v1.sch (EAGLE design)
At the start: 47 parts, among them IC2 FT230XS, IC3 AD708, IC4 LM2596S, Q2 PNP-TRANSISTIOR-2COLSOT89, X1 MINI-USB-32005-301

Commit message: Prawie done
Parts:
- added C10: 1uF, resistor:CPOL-EU085CS-1AW
- added R20: 10k, eagle-ltspice:RR3216
- added R21: 6k2, eagle-ltspice:RR3216
- C9: value 1u -> 2.2uF; device eagle-ltspice:C -> resistor:CPOL-EU085CS-1AW
Connections:
- removed net N$32: IC1.PA0
- removed net N$37: IC1.PA1
- new net N$41: IC1.PD1, R11.1
- new net N$42: IC1.PD0, R10.1
- new net N$44: IC1.PD4, R20.1, R21.1
- net GND: now also C10.-, C9.-, R20.2
- net N$15: now also C10.+
- net N$34: no longer C9.2
- net N$35: no longer C9.1
- net N$39: now also IC1.PA0
- net N$40: now also IC1.PA7; no longer IC1.PA5
- net VCC: now also C9.+, R21.2
Other:
- note added: "Todo: change ity"
- moved on the sheet: R18, R19

Commit message: Before ground wylawawing
Parts:
- added 0R: 6k2, eagle-ltspice:RR3216
Connections:
- new net R9: 0R.1
- net GND: now also 0R.2
Changed lines of the file:
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@@
 <part name="GND10" library="supply1" deviceset="GND" device="" value="GND D"/>
 <part name="SUPPLY17" library="supply2" deviceset="VCC" device="" value="VCC USB"/>
+<part name="GND11" library="supply1" deviceset="GND" device="" value="GND A"/>
+<part name="GND12" library="supply1" deviceset="GND" device="" value="GND D"/>
+<part name="0R" library="eagle-ltspice" deviceset="R" device="R3216" value="6k2"/>
 </parts>
 <sheets>
@@
 <instance part="GND10" gate="1" x="109.22" y="142.24"/>
 <instance part="SUPPLY17" gate="G$1" x="109.22" y="177.8"/>
+<instance part="GND11" gate="1" x="139.7" y="167.64"/>
+<instance part="GND12" gate="1" x="160.02" y="167.64"/>
+<instance part="0R" gate="G$1" x="149.86" y="182.88" rot="R180"/>
 </instances>
 <busses>
@@
 <wire x1="109.22" y1="144.78" x2="109.22" y2="147.32" width="0.1524" layer="91"/>
 </segment>
+<segment>
+<pinref part="0R" gate="G$1" pin="2"/>
+<pinref part="GND11" gate="1" pin="GND"/>
+<wire x1="144.78" y1="182.88" x2="139.7" y2="182.88" width="0.1524" layer="91"/>
+<wire x1="139.7" y1="182.88" x2="139.7" y2="170.18" width="0.1524" layer="91"/>
+</segment>
 </net>
 <net name="N$6" class="0">
@@
 </segment>
 </net>
+<net name="R9" class="0">
+<segment>
+<pinref part="0R" gate="G$1" pin="1"/>
+<pinref part="GND12" gate="1" pin="GND"/>
+<wire x1="154.94" y1="182.88" x2="160.02" y2="182.88" width="0.1524" layer="91"/>
+<wire x1="160.02" y1="182.88" x2="160.02" y2="170.18" width="0.1524" layer="91"/>
+</segment>
+</net>
