File: COdetector_pcb/PCB_v1.sch (EAGLE design)
At the start: 51 parts, among them IC2 FT230XS, IC3 AD708, IC4 LM2596S, Q2 PNP-TRANSISTIOR-2COLSOT89, X1 MINI-USB-32005-301

Commit message: V3 RC
Parts:
- removed LED1: TX, eagle-ltspice:LED_E
- removed LED2: RX, eagle-ltspice:LED_E
- removed R10, R9: 270R, eagle-ltspice:RR3216
- removed U$3: AVR-PDIHORZ, atmega-atxmega:AVR-PDIHORZ
- added PROG: (no value), con-lstb:MA03-1
- added SENSOR: (no value), con-lstb:MA06-1
- C8: value 100n -> 1u
- renumbered IC4 to LP2980, R11 to R5
Connections:
- removed net N$23: LED2.C, R9.1
- net GND: now also PROG.1, SENSOR.5; no longer C8.2, LED3.C, U$3.6
- net N$11: now also PROG.3; no longer U$3.1
- net N$12: now also PROG.2; no longer U$3.5
- net N$15: now also IC1.PA1, SENSOR.1; no longer C10.+, D1.C, D2.C, LP2980.!ON!/OFF, LP2980.VIN
- net N$20: now also IC1.PA2, SENSOR.2; no longer LED1.C, R8.1
- net N$21: now also IC1.PA3, SENSOR.3; no longer IC2.CBUS3, R8.2
- net N$22: now also IC1.PA4, SENSOR.4; no longer IC2.CBUS0, R9.2
- net N$26: now also LED3.C, R8.1; no longer LED3.A, R10.2
- net N$34: now also C8.2
- net N$35: now also C8.1
- net N$40: now also IC1.PA6; no longer IC1.PA7
- net N$42: now also IC1.PA7, R8.2; no longer IC1.PD0, R10.1
- net VCC: now also C10.+, D1.C, D2.C, LED3.A, LP2980.!ON!/OFF, LP2980.VIN, SENSOR.6; no longer C8.1, LED1.A, LED2.A, U$3.2
Other:
- note added: "To detect connected USB"
- note added: "Wrong pinout"
- note removed: "Todo: change ity"
- moved on the sheet: C4, C5, C6, C7, C8, IC2, IC3, L2, LED3, R12, R13, R14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

Commit message: Before sec version with all put togehter
Parts:
- removed IC3: AD708, ic-package:DIL8
- removed R14: 1k, pot-vitrohm:PC25
- removed R15: 1k, eagle-ltspice:RR3216
- removed R16, R18: 47k, eagle-ltspice:RR3216
- removed R17, R19: 180k, eagle-ltspice:RR3216
- C8: value 1u -> 100n
- R11: value 6k2 -> 5k6
- R12: value 1M -> 47k
- R13: value 2k -> 180k
- R2, R3: value 10k -> 27R
- R9: value 6k2 -> 0
- renumbered 0R to R9, LP2980 to LDO, R20 to R10, R21 to R11
Connections:
- removed net N$2: 3310.RESET, IC1.PC0
- removed net N$29: R12.2, R14.A
- removed net N$33: R13.1, R14.S
- removed net N$34: C8.2, IC3.1, R13.2, R17.1
- removed net N$35: C8.1, IC3.2, R12.1
- removed net N$36: R16.1, R17.2
- net GND: now also C8.2, R12.2; no longer IC3.3, IC3.4, IC3.5, IC3.6, R15.1, R15.2, R16.2, R18.2
- net N$15: now also 3310.RESET; no longer SENSOR.1
- net N$22: now also C8.1
- net N$25: no longer IC1.PD7
- net N$39: now also R12.1, R13.2; no longer R18.1, R19.2
- net VCC: now also R13.1; no longer IC3.8, R19.1
Other:
- note added: "TODO: increasew vals"
- moved on the sheet: C8, R12, R13
