File: COdetector_pcb/COdetector_pcb.brd (EAGLE design)
At the start: 35 parts

Commit message: Prawie done
Parts:
- removed C8: (no value), ref-packages:C0805K
- added E$3: (no value), pinhead:1X03/90
- added E$7: (no value), pinhead:1X02/90
- added R18, R20, R21: (no value), ref-packages:C0805K
- added R19: (no value), ref-packages-longpad:C1206K
- E$6: device atmega-atxmega:AVR-ISP-6 -> pinhead:1X06/90
- moved D2 39.0 mm to (66.0, 3.49)
- moved E$6 32.5 mm to (29.5, 36.5), turned to 90 degrees
- moved C6 15.5 mm to (81.6, 3.17), turned to 90 degrees
- moved C9 14.3 mm to (28.1, 5.65), turned to 0 degrees
- moved R8 11.2 mm to (49.2, 47.3), turned to 270 degrees
- moved L1 7.63 mm to (40.0, 44.1), turned to 180 degrees
- moved C10 7.25 mm to (29.2, 14.9)
- moved R4 7.03 mm to (46.0, 47.3)
- moved C5 6.96 mm to (74.6, 11.4), turned to 180 degrees
- moved IC4 5.99 mm to (26.0, 11.4)
- moved E$8 5.85 mm to (76.8, 41.0)
- moved Q1 5.75 mm to (71.1, 32.7)
- moved R5 5.75 mm to (67.3, 32.7)
- moved C1 4.50 mm to (42.4, 38.8), turned to 180 degrees
- moved E$1 4.49 mm to (76.2, 52.1)
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Connections:
- net S$41 renamed S$76
- net S$62 renamed S$74
- net S$69 renamed S$81
- removed net S$37: C3.1, C7.2, E$2.P08, E$2.P18, E$4.M1, E$4.M2, E$4.M3, E$4.M4
- removed net S$43: E$2.P17
- removed net S$50: E$8.+
- new net S$14: E$3.3
- new net S$61: E$2.P16, E$6.6
- new net S$70: E$1.K
- new net S$73: C3.1, C7.2, E$2.P08, E$2.P18, E$3.1, E$4.M1, E$4.M2, E$4.M3, E$4.M4, E$7.2
- new net S$78: E$6.3
- new net S$79: E$6.4
- new net S$80: E$7.1, E$8.+
- net S$38: now also E$3.2; no longer E$2.P16
- net S$56: no longer E$1.K
- net S$60: no longer E$6.6
Routing:
- net S$80: track 0.00 -> 122.0 mm
- net S$50: track 101.0 -> 0.45 mm
- net S$61: track 1.59 -> 95.3 mm
- net S$56: track 44.9 -> 3.49 mm
- net S$67: track 0.00 -> 35.6 mm
- net S$70: track 0.00 -> 34.2 mm
- net S$46: track 31.6 -> 0.00 mm
- net S$76: track 34.8 -> 10.5 mm
- net S$40: track 3.81 -> 27.6 mm
- net S$30: track 2.86 -> 26.5 mm
- net S$74: track 45.1 -> 23.4 mm
- net S$20: track 72.0 -> 53.7 mm
- net S$44: track 19.4 -> 3.17 mm
- net S$71: track 0.00 -> 15.1 mm
- net S$53: track 6.67 -> 20.4 mm
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Other:
- board text added: "3V3"
- board text removed: "Sprawdzic, gdzie masy!"

Commit message: Before ground wylawawing
Parts:
- removed E$1: (no value), led:LED5MM
- removed E$4: (no value), con-hirose:UX60A-MB-5ST
- removed E$8: (no value), buzzer:F/CM12P
- added BUZ: (no value), buzzer:F/CM12P
- added J0: (no value), ref-packages-longpad:C1206K
- added R9: (no value), ref-packages:C0805K
- added STAT: (no value), led:LED5MM
- added USB: (no value), con-hirose:UX60A-MB-5ST
- R3: device ref-packages:C0805K -> ref-packages-longpad:C1206K
- moved D1 35.3 mm to (25.7, 39.4)
- moved D2 23.3 mm to (79.1, 22.9), turned to 0 degrees
- moved C6 16.2 mm to (65.4, 3.81)
- moved L2 13.2 mm to (75.9, 27.6), turned to 0 degrees
- moved R5 9.96 mm to (58.1, 36.5), turned to 180 degrees
- moved Q1 9.16 mm to (63.5, 37.8)
- moved R7 9.16 mm to (63.5, 33.3)
- moved IC2 8.99 mm to (67.9, 26.4)
- moved C7 8.38 mm to (67.9, 31.8)
- moved R6 8.13 mm to (62.9, 29.5)
- moved R2 7.31 mm to (67.9, 19.7), turned to 0 degrees
- moved R3 4.85 mm to (74.6, 19.7), turned to 0 degrees
- moved C5 4.14 mm to (72.4, 14.9)
- moved C4 3.62 mm to (77.5, 14.9)
- moved R19 3.49 mm to (27.9, 24.8)
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- renumbered E$3 to PROG, E$6 to SENS, E$7 to BATT
Connections:
- removed net S$61: E$2.P16, SENS.6
- removed net S$63: E$8.-
- removed net S$73: BATT.2, C3.1, C7.2, E$2.P08, E$2.P18, E$4.M1, E$4.M2, E$4.M3, E$4.M4, PROG.1
- removed net S$74: SENS.5
- removed net S$80: BATT.1, E$8.+
- new net S$27: BUZ.-
- new net S$31: BATT.1
- new net S$35: SENS.6
- new net S$41: E$2.P16
- new net S$44: BUZ.+
- new net S$53: E$2.P07
- new net S$66: BATT.2, C3.1, C7.2, E$2.P08, E$2.P18, PROG.1, USB.M1, USB.M2, USB.M3, USB.M4
- net S$55: now also SENS.5; no longer E$2.P07
- net S$70: now also STAT.K; no longer E$1.K
- net S$81: now also STAT.A; no longer E$1.A
Routing:
- net S$66: track 2.86 -> 124.0 mm
- net S$80: track 122.0 -> 15.2 mm
- net S$61: track 95.3 -> 39.4 mm
- net S$44: track 3.17 -> 56.9 mm
- net S$20: track 53.7 -> 7.30 mm
- net S$41: track 1.40 -> 47.6 mm
- net S$74: track 23.4 -> 65.7 mm
- net S$73: track 7.27 -> 40.4 mm
- net S$35: track 6.16 -> 36.2 mm
- net S$55: track 4.45 -> 30.3 mm
- net S$30: track 26.5 -> 1.90 mm
- net S$40: track 27.6 -> 5.93 mm
- net S$29: track 2.99 -> 22.2 mm
- net S$53: track 20.4 -> 4.84 mm
- net S$84: track 0.00 -> 13.8 mm
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Other:
- board text added: "+"
- board text added: "-"
- board text added: "1"
- board text added: "11"
- board text added: "2015"
- board text added: "6"
- board text added: "A.Tyran"
- board text added: "Batt"
- board text added: "CO detector"
- board text removed: "3V3"
- board text removed: "Patrze od tyłu!"

Commit message: Super duper
Parts:
- R2: device ref-packages:C0805K -> rcl:C1206K
- moved C6 14.4 mm to (77.8, 11.1), turned to 180 degrees
- moved D2 5.12 mm to (79.7, 17.8), turned to 180 degrees
- moved R2 4.41 mm to (70.2, 15.9)
- moved L2 3.86 mm to (76.5, 23.8)
- moved C4 3.62 mm to (74.6, 17.1), turned to 90 degrees
- moved R3 3.13 mm to (71.8, 21.0), turned to 90 degrees
- moved R21 2.88 mm to (68.3, 12.1), turned to 90 degrees
- moved R5 2.54 mm to (58.1, 34.0)
- moved C5 2.48 mm to (74.3, 13.3)
- moved R1 2.22 mm to (41.6, 20.3)
- moved R20 1.59 mm to (65.1, 10.5)
- moved C1 1.09 mm to (43.3, 38.2)
- moved C2 0.91 mm to (43.3, 35.3)
- moved C9 0.78 mm to (27.8, 6.42), turned to 180 degrees
- moved D1 0.71 mm to (25.4, 40.0)
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Connections:
- removed net S$38: PROG.2
- removed net S$44: BUZ.+
- removed net S$66: BATT.2, C3.1, C7.2, E$2.P08, E$2.P18, PROG.1, USB.M1, USB.M2, USB.M3, USB.M4
- removed net S$81: STAT.A
- new net GNDD: BATT.2, C3.1, C7.2, C9.2, E$2.P08, E$2.P18, J0.1, PROG.1, USB.M1, USB.M2, USB.M3, USB.M4
- new net S$19: STAT.A
- new net S$7: PROG.2
Routing:
- net GNDD: track 0.00 -> 251.1 mm, vias 0 -> 4
- net S$66: track 124.0 -> 11.3 mm
- net S$74: track 65.7 -> 0.00 mm
- net S$30: track 1.90 -> 55.8 mm
- net S$61: track 39.4 -> 0.00 mm
- net S$67: track 35.3 -> 0.00 mm
- net S$81: track 25.1 -> 0.00 mm
- net S$19: track 2.85 -> 26.9 mm
- net S$44: track 56.9 -> 38.7 mm
- net S$80: track 15.2 -> 0.00 mm
- net S$84: track 13.8 -> 0.00 mm
- net S$59: track 17.0 -> 4.59 mm
- net S$6: track 39.7 -> 28.7 mm
- net S$20: track 7.30 -> 0.00 mm
- net S$25: track 5.15 -> 10.6 mm
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- added copper zone on layer 1, net GNDD

Commit message: Ready for first probe of make
Parts:
- moved C6 3.18 mm to (77.8, 14.3)
- moved BUZ 2.22 mm to (76.2, 38.7)
- moved R7 1.59 mm to (63.5, 34.9)
- moved R2 1.42 mm to (68.9, 15.2)
- moved R21 1.42 mm to (67.0, 11.4), turned to 270 degrees
- moved C5 1.31 mm to (74.0, 12.1)
- moved R20 1.00 mm to (64.8, 11.4)
- moved D1 0.95 mm to (26.4, 40.0)
- moved R18 0.95 mm to (29.5, 29.5)
- moved STAT 0.95 mm to (75.9, 49.5)
- moved R8 0.90 mm to (48.6, 47.9)
- moved R6 0.71 mm to (62.2, 29.8)
- moved R3 0.71 mm to (71.4, 20.3)
- moved R4 0.64 mm to (46.0, 47.9)
- moved D2 0.63 mm to (79.7, 18.4)
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Connections:
- net S$27 renamed S$20
- removed net GNDD: BATT.2, C3.1, C7.2, C9.2, E$2.P08, E$2.P18, J0.1, PROG.1, USB.M1, USB.M2, USB.M3, USB.M4
- new net GND: BATT.2, C10.1, C3.1, C4.1, C5.1, C6.2, C7.2, E$2.P08, E$2.P18, J0.1, J0.2, PROG.1, Q1.2, R7.1, R9.2, USB.5, USB.M1, USB.M2, USB.M3, USB.M4
- new net S$44: BUZ.+
Routing:
- net GND: track 0.00 -> 263.7 mm, vias 0 -> 4
- net GNDD: track 251.1 -> 0.00 mm, vias 4 -> 0
- net S$8: track 0.00 -> 3.91 mm
- net S$65: track 3.78 -> 0.00 mm
- net S$29: track 24.8 -> 21.3 mm
- net S$44: track 38.7 -> 35.5 mm
- net S$33: track 4.39 -> 1.51 mm
- net S$34: track 2.86 -> 0.00 mm
- net S$23: track 0.00 -> 2.22 mm
- net S$20: track 7.06 -> 8.97 mm
- net S$61: track 0.00 -> 1.91 mm
- net S$62: track 0.64 -> 2.30 mm
- net S$71: track 12.8 -> 14.4 mm
- net S$68: track 11.9 -> 13.5 mm
- net S$19: track 26.9 -> 28.4 mm
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- added copper zone on layer 1, net GND
- added copper zone on layer 1, net S$34
- added copper zone on layer 1, net S$50
- added copper zone on layer 1, net S$54
- added copper zone on layer 1, net S$65
- added copper zone on layer 1, net S$67
- added copper zone on layer 1, net S$74
- added copper zone on layer 1, net S$80
- added copper zone on layer 1, net S$81
- added copper zone on layer 1, net S$82
- added copper zone on layer 1, net S$83
- removed copper zone on layer 1, net GNDD
Other:
- board text removed: "+"
- board text removed: "-"
- board text removed: "1"
- board text removed: "11"
- board text removed: "6"
- board text removed: "Batt"

Commit message: Doone, checked, ready
Parts:
- moved D1 20.0 mm to (25.4, 20.0)
- moved C9 8.94 mm to (30.5, 14.6), turned to 90 degrees
- moved C10 8.67 mm to (26.4, 6.99), turned to 180 degrees
- moved R5 4.14 mm to (54.0, 34.3)
- moved R18 2.56 mm to (29.8, 32.1)
- moved R1 1.59 mm to (40.3, 19.4), turned to 0 degrees
- moved R19 1.59 mm to (27.9, 26.4)
- moved C3 0.90 mm to (55.2, 22.0)
- moved C2 0.71 mm to (43.0, 34.6)
- moved STAT 0.64 mm to (76.5, 49.5)
- moved R7 0.63 mm to (63.5, 34.3)
- moved C4 0.45 mm to (74.6, 17.5)
- moved R21 0.45 mm to (67.3, 11.7)
- moved R8 0.32 mm to (48.9, 47.9)
- moved R2 0.32 mm to (68.9, 15.6)
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Connections:
- new net S$81: C2.1, C2.2
- net GND: now also C9.1, R20.1; no longer C10.1, Q1.2
Routing:
- net S$73: track 40.1 -> 13.5 mm
- net S$31: track 10.0 -> 30.6 mm
- net S$86: track 0.00 -> 15.5 mm
- net S$57: track 15.5 -> 0.09 mm
- net GND: track 263.7 -> 275.4 mm, vias 4 -> 0
- net S$64: track 10.2 -> 17.5 mm
- net S$8: track 3.91 -> 0.00 mm
- net S$74: track 0.00 -> 2.80 mm
- net S$3: track 13.4 -> 11.0 mm
- net S$55: track 30.3 -> 28.0 mm
- net S$62: track 2.30 -> 0.00 mm, vias 0 -> 1
- net S$9: track 2.74 -> 4.57 mm
- net S$1: track 10.5 -> 8.77 mm
- net S$2: track 12.1 -> 10.4 mm
- net S$28: track 6.11 -> 4.52 mm
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- added copper zone on layer 1, net S$8
- added copper zone on layer 1, net S$84
- added copper zone on layer 1, net S$87
- added copper zone on layer 1, net S$88
- removed copper zone on layer 1, net S$74
- removed copper zone on layer 1, net S$81
- removed copper zone on layer 1, net S$83

Commit message: V3 RC
Parts:
- added .: (no value), pinhead:1X02/90
- added C8: (no value), ref-packages:C0805K
- C10, R18: device ref-packages:C0805K -> ref-packages:C1206K
- R19: device ref-packages-longpad:C1206K -> ref-packages:C1206K
- moved C6 22.8 mm to (58.4, 25.7)
- moved C3 22.7 mm to (33.9, 29.9)
- moved R18 22.1 mm to (8.25, 36.8), turned to 0 degrees
- moved BATT 21.6 mm to (9.84, 58.1)
- moved R3 21.3 mm to (50.8, 25.7)
- moved C10 21.3 mm to (6.03, 13.3)
- moved C7 20.8 mm to (48.3, 38.5), turned to 90 degrees
- moved C2 20.7 mm to (23.1, 40.3), turned to 0 degrees
- moved L2 20.7 mm to (56.8, 30.2)
- moved C9 20.7 mm to (10.8, 21.0)
- moved IC1 20.7 mm to (26.9, 33.5)
- moved PROG 20.7 mm to (9.84, 28.9)
- moved R19 20.7 mm to (8.26, 32.7)
- moved R6 20.7 mm to (42.2, 36.2)
- moved S1 20.7 mm to (14.9, 12.1)
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Connections:
- removed net S$20: BUZ.-
- removed net S$35: SENS.6
- removed net S$55: SENS.5
- removed net S$70: STAT.K
- removed net S$76: SENS.1
- removed net S$78: SENS.3
- removed net S$79: SENS.4
- new net S$36: SENS.2
- new net S$50: SENS.3
- new net S$54: SENS.4
- new net S$64: BUZ.-
- new net S$69: IC2.13
- net GND: now also ..2, Q1.2
- net S$31: now also SENS.5; no longer BATT.1
- net S$56: now also STAT.K; no longer E$2.P06
Routing:
- net GNDA: track 0.00 -> 38.9 mm
- net S$56: track 3.49 -> 40.0 mm
- net S$28: track 4.52 -> 37.1 mm
- net S$63: track 4.13 -> 36.0 mm
- net S$55: track 28.0 -> 0.12 mm
- net S$35: track 36.2 -> 10.7 mm
- net S$70: track 33.3 -> 13.4 mm
- net S$99: track 0.00 -> 17.8 mm
- net S$89: track 0.00 -> 17.0 mm
- net S$96: track 0.00 -> 15.5 mm
- net S$31: track 30.6 -> 46.0 mm
- net S$54: track 0.00 -> 15.3 mm
- net S$6: track 27.7 -> 13.2 mm
- net S$50: track 0.00 -> 14.0 mm
- net S$86: track 15.5 -> 29.1 mm
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- removed copper zone on layer 1, net S$34
- removed copper zone on layer 1, net S$50
- removed copper zone on layer 1, net S$54
- removed copper zone on layer 1, net S$65
- removed copper zone on layer 1, net S$67
- removed copper zone on layer 1, net S$8
- removed copper zone on layer 1, net S$82
- removed copper zone on layer 1, net S$84
- removed copper zone on layer 1, net S$87
- removed copper zone on layer 1, net S$88

Commit message: Before sec version with all put togehter
Parts:
- moved C10 0.64 mm to (6.03, 12.7)
- flipped S1 to the top
- flipped S2 to the top
- flipped S3 to the top
- renumbered IC4 to LDO, R18 to R12, R19 to R13, R20 to R10, R21 to R11
Routing:
- net GND: track 282.0 -> 278.3 mm
- net S$85: track 0.00 -> 3.01 mm
- net S$63: track 36.0 -> 35.3 mm
- net S$87: track 0.00 -> 0.58 mm

Commit message: New Version, final
Parts:
- removed ., BATT: (no value), pinhead:1X02/90
- removed D1: (no value), rcl:M1206
- removed J0: (no value), ref-packages-longpad:C1206K
- removed L1, L2: (no value), ref-packages:C1812K
- removed PROG: (no value), pinhead:1X03/90
- removed Q2: (no value), avago:SOT23
- removed SENS: (no value), pinhead:1X06/90
- added C11, J1: (no value), ref-packages:C1206K
- added C12, C13, R14, R15: (no value), ref-packages:C0805K
- added E$1: (no value), battery:SL-160AA/PR
- added E$10: (no value), con-lstb:MA03-1
- added E$3: (no value), discrete:R-7,5
- added E$4: (no value), atmel:8S1
- added E$5: (no value), pot:B64Y
- added E$6: (no value), ref-packages:0207/10
- added E$7: (no value), pinhead:1X02
- added E$8: (no value), diode:DO34Z7
- added E$9: (no value), ref-packages:TO92-LINE
- added J2: (no value), ref-packages-longpad:C1206K
- E$2: device 3310LCD:3310 -> con-lstb:MA08-1
- moved E$2 23.4 mm to (39.7, 21.6)
- moved R8 20.4 mm to (45.7, 41.6), turned to 0 degrees
- moved R12 18.5 mm to (23.5, 26.4), turned to 90 degrees
- moved C10 14.4 mm to (20.3, 11.1), turned to 270 degrees
- moved D2 13.8 mm to (73.7, 10.5)
- moved USB 13.0 mm to (66.0, 4.45)
- moved C8 12.7 mm to (32.7, 38.6), turned to 90 degrees
- moved C3 12.7 mm to (46.6, 29.3)
- moved C5 12.7 mm to (68.0, 18.4)
- moved IC1 12.7 mm to (39.6, 32.9)
- moved IC2 12.7 mm to (61.0, 32.1)
- moved R10 12.7 mm to (59.4, 13.7)
- moved R11 12.7 mm to (62.5, 13.7)
- moved R2 12.7 mm to (61.9, 20.0)
- moved R3 12.7 mm to (63.5, 25.1)
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Connections:
- removed net S$14: PROG.3
- removed net S$19: STAT.A
- removed net S$2: E$2.P12
- removed net S$3: E$2.P11
- removed net S$31: SENS.5
- removed net S$36: SENS.2
- removed net S$4: E$2.P15
- removed net S$41: E$2.P16
- removed net S$5: E$2.P14
- removed net S$50: SENS.3
- removed net S$53: E$2.P07
- removed net S$64: BUZ.-
- removed net S$7: PROG.2
- removed net S$81: C2.1, C2.2
- new net S$102: E$3.1
- new net S$106: E$10.3
- new net S$108: E$8.C
- new net S$111: R10.1
- new net S$18: E$6.2
- new net S$22: E$3.2
- new net S$55: STAT.A
- new net S$57: E$2.3
- new net S$62: E$9.1, STAT.K
- new net S$71: E$5.S
- new net S$8: Q1.2
- new net S$84: E$6.1
- new net S$86: E$9.2
- net GND: now also C1.1, E$1.-, E$10.1, E$2.8, E$5.E, E$7.1, E$9.3, J2.1, J2.2, R12.1; no longer ..2, BATT.2, E$2.P08, E$2.P18, J0.1, J0.2, PROG.1, Q1.2, R10.1
- net S$1: now also C2.1, C2.2; no longer E$2.P13
- net S$44: now also E$5.A; no longer BUZ.+
- net S$54: now also E$7.2, E$8.A; no longer SENS.4
- net S$56: now also BUZ.-; no longer STAT.K
Routing:
- net GND: track 278.3 -> 375.4 mm, vias 9 -> 0
- net S$62: track 0.00 -> 68.9 mm, vias 1 -> 0
- net S$108: track 0.00 -> 63.3 mm
- net S$30: track 58.1 -> 2.88 mm
- net S$54: track 15.3 -> 62.1 mm
- net S$31: track 46.0 -> 2.86 mm
- net S$84: track 1.14 -> 41.7 mm
- net GNDA: track 38.9 -> 0.00 mm
- net S$19: track 31.6 -> 0.00 mm
- net S$56: track 40.0 -> 8.77 mm
- net S$100: track 0.00 -> 29.4 mm
- net S$63: track 35.3 -> 7.80 mm, vias 0 -> 2
- net S$55: track 0.12 -> 27.5 mm
- net S$86: track 29.1 -> 4.20 mm
- net S$88: track 0.00 -> 21.2 mm
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- added copper zone on layer 1, net S$76
- added copper zone on layer 1, net S$83
Other:
- board text added: "CO MONITOR by A. Tyran AGH WIEiT Kraków 2015"
- board text added: "TGS5042"
- board text removed: "2015"
- board text removed: "A.Tyran"
- board text removed: "CO detector"
